Commit message: working servo demo

File: urdf/test_bench.urdf.xacro (robot description, xacro)
@@ -1,10 +1,30 @@
 <?xml version="1.0"?>
 <robot xmlns:xacro="http://www.ros.org/wiki/xacro" name="wisco_test_bench">
-  <link name="base_link"/>
-  <link name="test_mass"/>
+  <link name="base_link">
+    <visual>
+<origin xyz="0.01 0 0" rpy="0 0 0"/>
+      <geometry><cylinder radius="0.05" length="0.11"/></geometry>
+      <material name="black"><color rgba="0.1 0.1 0.1 1"/></material>
+    </visual>
+  </link>
+  <link name="test_mass">
+    <visual>
+      <!-- Main cylinder body -->
+      <origin xyz="0.01 0 0.01" rpy="0 0 0"/>
+      <geometry><cylinder radius="0.05" length="0.11"/></geometry>
+      <material name="red"><color rgba="1 0.2 0.2 1"/></material>
+    </visual>
+    <visual>
+      <!-- Asymmetric pointer box sticking out radially to show rotation -->
+      <origin xyz="0.05 0 0.07" rpy="0 0 0"/>
+      <geometry><box size="0.04 0.02 0.02"/></geometry>
+      <material name="red"><color rgba="1 1 1 1"/></material>
+    </visual>
+  </link>
   <joint name="test_motor_joint" type="continuous">
     <parent link="base_link"/>
     <child link="test_mass"/>
     <axis xyz="0 0 1"/>
+    <calibration rising = "0.0"/>
   </joint>
   <ros2_control name="EthercatTestBench" type="system">
@@ -12,19 +32,19 @@
       <plugin>ethercat_driver/EthercatDriver</plugin>
       <param name="master_id">0</param>
-      <param name="control_frequency">1000</param>
+      <param name="control_frequency">100</param>
     </hardware>
-    <joint name="test_motor_joint">
-      <state_interface name="position"/>
-      <state_interface name="velocity"/>
-      <state_interface name="effort"/>
-      <command_interface name="effort"/>
-      <command_interface name="reset_fault"/>
-      <ec_module name="rmd_test_motor">
-        <plugin>ethercat_generic_plugins/EcCiA402Drive</plugin>
-        <param name="alias">0</param>
-        <param name="position">0</param>
-        <param name="slave_config">$(find wisco_hw_interface)/config/rmd_x4_10.yaml</param>
-      </ec_module>
-    </joint>
-  </ros2_control>
+<joint name="test_motor_joint">
+  <state_interface name="position"/>
+  <state_interface name="velocity"/>
+  <state_interface name="effort"/>
+  <command_interface name="effort"/>
+  <command_interface name="reset_fault"/>
+  <ec_module name="rmd_test_motor">
+    <plugin>ethercat_generic_plugins/EcCiA402Drive</plugin>
+    <param name="alias">0</param>
+    <param name="position">0</param>
+    <param name="slave_config">$(find wisco_ethercat_ros2_hw)/config/rmd_x4_10.yaml</param>
+  </ec_module>
+</joint>
+ </ros2_control>
 </robot>

Commit message: added todos

File: urdf/test_bench.urdf.xacro (robot description, xacro)
@@ -1,50 +1,33 @@
 <?xml version="1.0"?>
-<robot xmlns:xacro="http://www.ros.org/wiki/xacro" name="wisco_test_bench">
-  <link name="base_link">
-    <visual>
-<origin xyz="0.01 0 0" rpy="0 0 0"/>
-      <geometry><cylinder radius="0.05" length="0.11"/></geometry>
-      <material name="black"><color rgba="0.1 0.1 0.1 1"/></material>
-    </visual>
-  </link>
-  <link name="test_mass">
-    <visual>
-      <!-- Main cylinder body -->
-      <origin xyz="0.01 0 0.01" rpy="0 0 0"/>
-      <geometry><cylinder radius="0.05" length="0.11"/></geometry>
-      <material name="red"><color rgba="1 0.2 0.2 1"/></material>
-    </visual>
-    <visual>
-      <!-- Asymmetric pointer box sticking out radially to show rotation -->
-      <origin xyz="0.05 0 0.07" rpy="0 0 0"/>
-      <geometry><box size="0.04 0.02 0.02"/></geometry>
-      <material name="red"><color rgba="1 1 1 1"/></material>
-    </visual>
-  </link>
-  <joint name="test_motor_joint" type="continuous">
-    <parent link="base_link"/>
-    <child link="test_mass"/>
-    <axis xyz="0 0 1"/>
-    <calibration rising = "0.0"/>
-  </joint>
-  <ros2_control name="EthercatTestBench" type="system">
+<robot xmlns:xacro="http://www.ros.org/wiki/xacro" name="multi_actuator_test_bench">
+  <!-- TODO(Multi-Actuator): Define links and joints for multi-actuator kinematic chain (e.g., shoulder, elbow, wrist) -->
+  <ros2_control name="EtherCATSystem" type="system">
     <hardware>
       <plugin>ethercat_driver/EthercatDriver</plugin>
       <param name="master_id">0</param>
-      <param name="control_frequency">100</param>
+      <!-- TODO(Multi-Actuator): Update EtherCAT loop rate and interface configurations -->
     </hardware>
-<joint name="test_motor_joint">
-  <state_interface name="position"/>
-  <state_interface name="velocity"/>
-  <state_interface name="effort"/>
-  <command_interface name="effort"/>
-  <command_interface name="reset_fault"/>
-  <ec_module name="rmd_test_motor">
-    <plugin>ethercat_generic_plugins/EcCiA402Drive</plugin>
-    <param name="alias">0</param>
-    <param name="position">0</param>
-    <param name="slave_config">$(find wisco_ethercat_ros2_hw)/config/rmd_x4_10.yaml</param>
-  </ec_module>
-</joint>
- </ros2_control>
+    <!-- TODO(Multi-Actuator): Add joint hardware definitions and EtherCAT slave indices (0, 1, 2) for each daisy-chained actuator -->
+    <joint name="joint_1">
+      <state_interface name="position"/>
+      <state_interface name="velocity"/>
+      <state_interface name="effort"/>
+      <command_interface name="effort"/>
+      <!-- TODO(Multi-Actuator): Map PDO parameters for Actuator 1 (Slave Index 0) -->
+    </joint>
+    <joint name="joint_2">
+      <state_interface name="position"/>
+      <state_interface name="velocity"/>
+      <state_interface name="effort"/>
+      <command_interface name="effort"/>
+      <!-- TODO(Multi-Actuator): Map PDO parameters for Actuator 2 (Slave Index 1) -->
+    </joint>
+    <joint name="joint_3">
+      <state_interface name="position"/>
+      <state_interface name="velocity"/>
+      <state_interface name="effort"/>
+      <command_interface name="effort"/>
+      <!-- TODO(Multi-Actuator): Map PDO parameters for Actuator 3 (Slave Index 2) -->
+    </joint>
+  </ros2_control>
 </robot>

Commit message: throwing stuff at the wall

File: urdf/test_bench.urdf.xacro (robot description, xacro)
@@ -2,4 +2,65 @@
 <robot xmlns:xacro="http://www.ros.org/wiki/xacro" name="multi_actuator_test_bench">
   <!-- TODO(Multi-Actuator): Define links and joints for multi-actuator kinematic chain (e.g., shoulder, elbow, wrist) -->
+  <joint name="shoulder_joint" type="revolute">
+    <parent link="base_link"/>
+    <child link="upper_arm_link"/>
+    <origin xyz="0 0 0" rpy="0 0 0"/>
+    <axis xyz="0 0 1"/>
+    <limit lower="-1.57" upper="1.57" effort="10" velocity="1.0"/>
+  </joint>
+  <joint name="elbow_joint" type="revolute">
+    <parent link="upper_arm_link"/>
+    <child link="forearm_link"/>
+    <origin xyz="0 0 0" rpy="0 0 0"/>
+    <axis xyz="0 1 0"/>
+    <limit lower="-1.57" upper="1.57" effort="10" velocity="1.0"/>
+  </joint>
+  <joint name="wrist_joint" type="revolute">
+    <parent link="forearm_link"/>
+    <child link="hand_link"/>
+    <origin xyz="0 0 0" rpy="0 0 0"/>
+    <axis xyz="1 0 0"/>
+    <limit lower="-1.57" upper="1.57" effort="10" velocity="1.0"/>
+  </joint>
+  link name="base_link">
+    <visual>
+      <geometry>
+        <box size="0.2 0.2 0.1"/>
+      </geometry>
+      <material name="gray">
+        <color rgba="0.5 0.5 0.5 1.0"/>
+      </material>
+    </visual>
+  </link>
+  link name="upper_arm_link">
+    <visual>
+      <geometry>
+        <cylinder length="0.3" radius="0.05"/>
+      </geometry>
+      <material name="blue">
+        <color rgba="0.0 0.0 1.0 1.0"/>
+      </material>
+    </visual>
+  </link>
+  link name="forearm_link">
+    <visual>
+      <geometry>
+        <cylinder length="0.25" radius="0.04"/>
+      </geometry>
+      <material name="green">
+        <color rgba="0.0 1.0 0.0 1.0"/>
+      </material>
+    </visual>
+  </link>
+  link name="hand_link">
+    <visual>
+      <geometry>
+        <box size="0.1 0.1 0.05"/>
+      </geometry>
+      <material name="red">
+        <color rgba="1.0 0.0 0.0 1.0"/>
+      </material>
+    </visual>
+  </link>
   <ros2_control name="EtherCATSystem" type="system">
     <hardware>
@@ -7,4 +68,8 @@
       <param name="master_id">0</param>
       <!-- TODO(Multi-Actuator): Update EtherCAT loop rate and interface configurations -->
+      <param name="loop_rate">1000</param>
+      <param name="interface_type">EtherCAT</param>
+      <param name="pdo_mapping">true</param>
+      <param name="slave_count">3</param>
     </hardware>
     <!-- TODO(Multi-Actuator): Add joint hardware definitions and EtherCAT slave indices (0, 1, 2) for each daisy-chained actuator -->
@@ -15,4 +80,21 @@
       <command_interface name="effort"/>
       <!-- TODO(Multi-Actuator): Map PDO parameters for Actuator 1 (Slave Index 0) -->
+      <ros2_control name="joint_1_controller" type="effort_controller/JointEffortController">
+        <param name="joint">joint_1</param>
+        <param name="command_topic">/joint_1/command</param>
+      </ros2_control>
+      <ros2_control name="joint_1_state_broadcaster" type="joint_state_broadcaster/JointStateBroadcaster">
+        <param name="joint">joint_1</param>
+        <param name="state_topic">/joint_1/state</param>
+      </ros2_control>
+      <ros2_control name="joint_1_safety_monitor" type="safety_monitor/SafetyMonitor">
+        <param name="joint">joint_1</param>
+        <param name="effort_limit">5.0</param>
+        <param name="velocity_limit">1.0</param>
+      </ros2_control>
+      <ros2_control name="joint_1_telemetry" type="telemetry/JointTelemetry">
+        <param name="joint">joint_1</param>
+        <param name="telemetry_topic">/joint_1/telemetry</param>
+      </ros2_control>
     </joint>
     <joint name="joint_2">
@@ -22,4 +104,20 @@
       <command_interface name="effort"/>
       <!-- TODO(Multi-Actuator): Map PDO parameters for Actuator 2 (Slave Index 1) -->
+              <param name="joint">joint_2</param>
+        <param name="command_topic">/joint_2/command</param>
+      </ros2_control>
+      <ros2_control name="joint_2_state_broadcaster" type="joint_state_broadcaster/JointStateBroadcaster">
+        <param name="joint">joint_2</param>
+        <param name="state_topic">/joint_2/state</param>
+      </ros2_control>
+      <ros2_control name="joint_2_safety_monitor" type="safety_monitor/SafetyMonitor">
+        <param name="joint">joint_2</param>
+        <param name="effort_limit">5.0</param>
+        <param name="velocity_limit">1.0</param>
+      </ros2_control>
+      <ros2_control name="joint_2_telemetry" type="telemetry/JointTelemetry">
+        <param name="joint">joint_2</param>
+        <param name="telemetry_topic">/joint_2/telemetry</param>
+      </ros2_control>
     </joint>
     <joint name="joint_3">
@@ -29,4 +127,20 @@
       <command_interface name="effort"/>
       <!-- TODO(Multi-Actuator): Map PDO parameters for Actuator 3 (Slave Index 2) -->
+      <param name="joint">joint_3</param>
+        <param name="command_topic">/joint_3/command</param>
+      </ros2_control>
+      <ros2_control name="joint_3_state_broadcaster" type="joint_state_broadcaster/JointStateBroadcaster">
+        <param name="joint">joint_3</param>
+        <param name="state_topic">/joint_3/state</param>
+      </ros2_control>
+      <ros2_control name="joint_3_safety_monitor" type="safety_monitor/SafetyMonitor">
+        <param name="joint">joint_3</param>
+        <param name="effort_limit">5.0</param>
+        <param name="velocity_limit">1.0</param>
+      </ros2_control>
+      <ros2_control name="joint_3_telemetry" type="telemetry/JointTelemetry">
+        <param name="joint">joint_3</param>
+        <param name="telemetry_topic">/joint_3/telemetry</param>
+      </ros2_control>
     </joint>
   </ros2_control>

Commit message: cleaned up some errors

File: urdf/test_bench.urdf.xacro (robot description, xacro)
@@ -1,5 +1,45 @@
 <?xml version="1.0"?>
 <robot xmlns:xacro="http://www.ros.org/wiki/xacro" name="multi_actuator_test_bench">
-  <!-- TODO(Multi-Actuator): Define links and joints for multi-actuator kinematic chain (e.g., shoulder, elbow, wrist) -->
+  <!-- Links -->
+  <link name="base_link">
+    <visual>
+      <geometry>
+        <box size="0.2 0.2 0.1"/>
+      </geometry>
+      <material name="gray">
+        <color rgba="0.5 0.5 0.5 1.0"/>
+      </material>
+    </visual>
+  </link>
+  <link name="upper_arm_link">
+    <visual>
+      <geometry>
+        <cylinder length="0.3" radius="0.05"/>
+      </geometry>
+      <material name="blue">
+        <color rgba="0.0 0.0 1.0 1.0"/>
+      </material>
+    </visual>
+  </link>
+  <link name="forearm_link">
+    <visual>
+      <geometry>
+        <cylinder length="0.25" radius="0.04"/>
+      </geometry>
+      <material name="green">
+        <color rgba="0.0 1.0 0.0 1.0"/>
+      </material>
+    </visual>
+  </link>
+  <link name="hand_link">
+    <visual>
+      <geometry>
+        <box size="0.1 0.1 0.05"/>
+      </geometry>
+      <material name="red">
+        <color rgba="1.0 0.0 0.0 1.0"/>
+      </material>
+    </visual>
+  </link>
   <joint name="shoulder_joint" type="revolute">
     <parent link="base_link"/>
@@ -23,49 +63,8 @@
     <limit lower="-1.57" upper="1.57" effort="10" velocity="1.0"/>
   </joint>
-  link name="base_link">
-    <visual>
-      <geometry>
-        <box size="0.2 0.2 0.1"/>
-      </geometry>
-      <material name="gray">
-        <color rgba="0.5 0.5 0.5 1.0"/>
-      </material>
-    </visual>
-  </link>
-  link name="upper_arm_link">
-    <visual>
-      <geometry>
-        <cylinder length="0.3" radius="0.05"/>
-      </geometry>
-      <material name="blue">
-        <color rgba="0.0 0.0 1.0 1.0"/>
-      </material>
-    </visual>
-  </link>
-  link name="forearm_link">
-    <visual>
-      <geometry>
-        <cylinder length="0.25" radius="0.04"/>
-      </geometry>
-      <material name="green">
-        <color rgba="0.0 1.0 0.0 1.0"/>
-      </material>
-    </visual>
-  </link>
-  link name="hand_link">
-    <visual>
-      <geometry>
-        <box size="0.1 0.1 0.05"/>
-      </geometry>
-      <material name="red">
-        <color rgba="1.0 0.0 0.0 1.0"/>
-      </material>
-    </visual>
-  </link>
   <ros2_control name="EtherCATSystem" type="system">
     <hardware>
       <plugin>ethercat_driver/EthercatDriver</plugin>
       <param name="master_id">0</param>
-      <!-- TODO(Multi-Actuator): Update EtherCAT loop rate and interface configurations -->
       <param name="loop_rate">1000</param>
       <param name="interface_type">EtherCAT</param>
@@ -73,74 +72,39 @@
       <param name="slave_count">3</param>
     </hardware>
-    <!-- TODO(Multi-Actuator): Add joint hardware definitions and EtherCAT slave indices (0, 1, 2) for each daisy-chained actuator -->
-    <joint name="joint_1">
+    <joint name="shoulder_joint">
       <state_interface name="position"/>
       <state_interface name="velocity"/>
       <state_interface name="effort"/>
       <command_interface name="effort"/>
-      <!-- TODO(Multi-Actuator): Map PDO parameters for Actuator 1 (Slave Index 0) -->
-      <ros2_control name="joint_1_controller" type="effort_controller/JointEffortController">
-        <param name="joint">joint_1</param>
-        <param name="command_topic">/joint_1/command</param>
-      </ros2_control>
-      <ros2_control name="joint_1_state_broadcaster" type="joint_state_broadcaster/JointStateBroadcaster">
-        <param name="joint">joint_1</param>
-        <param name="state_topic">/joint_1/state</param>
-      </ros2_control>
-      <ros2_control name="joint_1_safety_monitor" type="safety_monitor/SafetyMonitor">
-        <param name="joint">joint_1</param>
-        <param name="effort_limit">5.0</param>
-        <param name="velocity_limit">1.0</param>
-      </ros2_control>
-      <ros2_control name="joint_1_telemetry" type="telemetry/JointTelemetry">
-        <param name="joint">joint_1</param>
-        <param name="telemetry_topic">/joint_1/telemetry</param>
-      </ros2_control>
+      <ec_module name="shoulder_actuator">
+        <plugin>ethercat_generic_plugins/EcCiA402Drive</plugin>
+        <param name="alias">0</param>
+        <param name="position">0</param>
+        <param name="slave_id">0</param>
+      </ec_module>
     </joint>
-    <joint name="joint_2">
+    <joint name="elbow_joint">
       <state_interface name="position"/>
       <state_interface name="velocity"/>
       <state_interface name="effort"/>
       <command_interface name="effort"/>
-      <!-- TODO(Multi-Actuator): Map PDO parameters for Actuator 2 (Slave Index 1) -->
-              <param name="joint">joint_2</param>
-        <param name="command_topic">/joint_2/command</param>
-      </ros2_control>
-      <ros2_control name="joint_2_state_broadcaster" type="joint_state_broadcaster/JointStateBroadcaster">
-        <param name="joint">joint_2</param>
-        <param name="state_topic">/joint_2/state</param>
-      </ros2_control>
-      <ros2_control name="joint_2_safety_monitor" type="safety_monitor/SafetyMonitor">
-        <param name="joint">joint_2</param>
-        <param name="effort_limit">5.0</param>
-        <param name="velocity_limit">1.0</param>
-      </ros2_control>
-      <ros2_control name="joint_2_telemetry" type="telemetry/JointTelemetry">
-        <param name="joint">joint_2</param>
-        <param name="telemetry_topic">/joint_2/telemetry</param>
-      </ros2_control>
+      <ec_module name="elbow_actuator">
+        <plugin>ethercat_generic_plugins/EcCiA402Drive</plugin>
+        <param name="alias">0</param>
+        <param name="position">1</param>
+        <param name="slave_id">1</param>
+      </ec_module>
     </joint>
-    <joint name="joint_3">
+    <joint name="wrist_joint">
       <state_interface name="position"/>
       <state_interface name="velocity"/>
       <state_interface name="effort"/>
       <command_interface name="effort"/>
-      <!-- TODO(Multi-Actuator): Map PDO parameters for Actuator 3 (Slave Index 2) -->
-      <param name="joint">joint_3</param>
-        <param name="command_topic">/joint_3/command</param>
-      </ros2_control>
-      <ros2_control name="joint_3_state_broadcaster" type="joint_state_broadcaster/JointStateBroadcaster">
-        <param name="joint">joint_3</param>
-        <param name="state_topic">/joint_3/state</param>
-      </ros2_control>
-      <ros2_control name="joint_3_safety_monitor" type="safety_monitor/SafetyMonitor">
-        <param name="joint">joint_3</param>
-        <param name="effort_limit">5.0</param>
-        <param name="velocity_limit">1.0</param>
-      </ros2_control>
-      <ros2_control name="joint_3_telemetry" type="telemetry/JointTelemetry">
-        <param name="joint">joint_3</param>
-        <param name="telemetry_topic">/joint_3/telemetry</param>
-      </ros2_control>
+      <ec_module name="wrist_actuator">
+        <plugin>ethercat_generic_plugins/EcCiA402Drive</plugin>
+        <param name="alias">0</param>
+        <param name="position">2</param>
+        <param name="slave_id">2</param>
+      </ec_module>
     </joint>
   </ros2_control>

Commit message: test success

File: urdf/test_bench.urdf.xacro (robot description, xacro)
@@ -4,4 +4,5 @@
   <link name="base_link">
     <visual>
+      <origin xyz="0 0 0.05" rpy="0 0 0"/>
       <geometry>
         <box size="0.2 0.2 0.1"/>
@@ -13,5 +14,7 @@
   </link>
   <link name="upper_arm_link">
+    <!-- Main Arm Cylinder -->
     <visual>
+      <origin xyz="0 0 0.15" rpy="0 0 0"/>
       <geometry>
         <cylinder length="0.3" radius="0.05"/>
@@ -21,7 +24,18 @@
       </material>
     </visual>
+    <!-- Indicator box to show axial rotation -->
+    <visual>
+      <origin xyz="0.05 0 0.15" rpy="0 0 0"/>
+      <geometry>
+        <box size="0.05 0.02 0.02"/>
+      </geometry>
+      <material name="red">
+        <color rgba="1.0 0.0 0.0 1.0"/>
+      </material>
+    </visual>
   </link>
   <link name="forearm_link">
     <visual>
+      <origin xyz="0 0 0.125" rpy="0 0 0"/>
       <geometry>
         <cylinder length="0.25" radius="0.04"/>
@@ -34,4 +48,5 @@
   <link name="hand_link">
     <visual>
+      <origin xyz="0 0 0.025" rpy="0 0 0"/>
       <geometry>
         <box size="0.1 0.1 0.05"/>
@@ -42,8 +57,9 @@
     </visual>
   </link>
+  <!-- Joints -->
   <joint name="shoulder_joint" type="revolute">
     <parent link="base_link"/>
     <child link="upper_arm_link"/>
-    <origin xyz="0 0 0" rpy="0 0 0"/>
+    <origin xyz="0 0 0.1" rpy="0 0 0"/> <!-- Starts at top of base -->
     <axis xyz="0 0 1"/>
     <limit lower="-1.57" upper="1.57" effort="10" velocity="1.0"/>
@@ -52,5 +68,5 @@
     <parent link="upper_arm_link"/>
     <child link="forearm_link"/>
-    <origin xyz="0 0 0" rpy="0 0 0"/>
+    <origin xyz="0 0 0.3" rpy="0 0 0"/> <!-- Starts at end of upper arm -->
     <axis xyz="0 1 0"/>
     <limit lower="-1.57" upper="1.57" effort="10" velocity="1.0"/>
@@ -59,8 +75,9 @@
     <parent link="forearm_link"/>
     <child link="hand_link"/>
-    <origin xyz="0 0 0" rpy="0 0 0"/>
+    <origin xyz="0 0 0.25" rpy="0 0 0"/> <!-- Starts at end of forearm -->
     <axis xyz="1 0 0"/>
     <limit lower="-1.57" upper="1.57" effort="10" velocity="1.0"/>
   </joint>
+  <!-- ros2_control definition remains exactly the same -->
   <ros2_control name="EtherCATSystem" type="system">
     <hardware>
@@ -82,4 +99,5 @@
         <param name="position">0</param>
         <param name="slave_id">0</param>
+        <param name="slave_config">$(find wisco_ethercat_ros2_hw)/config/rmd_x4_10.yaml</param>
       </ec_module>
     </joint>
@@ -94,4 +112,5 @@
         <param name="position">1</param>
         <param name="slave_id">1</param>
+        <param name="slave_config">$(find wisco_ethercat_ros2_hw)/config/rmd_x4_10.yaml</param>
       </ec_module>
     </joint>
@@ -106,4 +125,5 @@
         <param name="position">2</param>
         <param name="slave_id">2</param>
+        <param name="slave_config">$(find wisco_ethercat_ros2_hw)/config/rmd_x4_10.yaml</param>
       </ec_module>
     </joint>
